Commit message: Change robot 1 color to purple
Co-authored-by: Giovanni Lorenzini <giovanni@lorenzinigiovanni.com>
Co-authored-by: Diego Planchenstainer <d.planchenstainer@studenti.unitn.it>

File: src/0_mindstorm_simulator/1_lego_robot/urdf/my_robot_1.xacro (robot description, xacro)
@@ -210,5 +210,5 @@
 </gazebo>
 <gazebo reference="top_triangle">
-    <material>Gazebo/Yellow</material>
+    <material>Gazebo/Purple</material>
 </gazebo>
 <gazebo reference="top_layer">
